Commit message: intrepid description: changed urdf robot name to intrepid + modified lidar location + removed GPS (until actual location is known)

File: intrepid_description/urdf/robots/intrepid.urdf.xacro (robot description, xacro)
@@ -1,5 +1,5 @@
 <?xml version="1.0"?>
 <!-- rbvogui v3.0 -->
-<robot name="rbvogui" xmlns:xacro="http://www.ros.org/wiki/xacro">
+<robot name="intrepid" xmlns:xacro="http://www.ros.org/wiki/xacro">
     <!-- ***************** -->
     <!-- Imported elements -->
@@ -28,7 +28,11 @@
     <xacro:property name="rocker_offset_z" value="0.130" />
     <!-- RS-Lidar -->
-    <xacro:property name="top_lidar_offset_x" value="0.343" />
+<!--     <xacro:property name="top_lidar_offset_x" value="0.343" />
     <xacro:property name="top_lidar_offset_y" value="0.0" />
     <xacro:property name="top_lidar_offset_z" value="1.302" />
+ -->
+    <xacro:property name="top_lidar_offset_x" value="0.260" />
+    <xacro:property name="top_lidar_offset_y" value="0.0" />
+    <xacro:property name="top_lidar_offset_z" value="0.606" />
     <!-- Basket parameters -->
     <xacro:property name="basket_offset_x" value="0.0" />
@@ -45,5 +49,5 @@
     <xacro:arg name="prefix" default="robot_" />
     <xacro:property name="gpu" default="false" />
-    <xacro:macro name="rbvogui" params="prefix publish_bf hq gpu">
+    <xacro:macro name="intrepid" params="prefix publish_bf hq gpu">
         <!-- *************** -->
         <!-- Robots Elements -->
@@ -85,7 +89,7 @@
         </xacro:sensor_imu_hector>
         <!-- GPS -->
-        <xacro:sensor_gps prefix="${prefix}gps" parent="${prefix}base_link">
+<!--         <xacro:sensor_gps prefix="${prefix}gps" parent="${prefix}base_link">
             <origin xyz="0.344 -0.128 1.212" rpy="0 0 0"/>
-        </xacro:sensor_gps>
+        </xacro:sensor_gps> -->
         <!-- RS-Lidar -->
         <xacro:sensor_rslidar_16 prefix="${prefix}top_3d_laser" parent="${prefix}base_link" prefix_topic="top_3d_laser" gpu="${gpu}">
@@ -102,4 +106,4 @@
     <!-- Gazebo ros control pluggins -->
     <xacro:ros_control/>
-    <xacro:rbvogui prefix="$(arg prefix)" publish_bf="${publish_bf}" hq="${hq}" gpu="${gpu}"/>
+    <xacro:intrepid prefix="$(arg prefix)" publish_bf="${publish_bf}" hq="${hq}" gpu="${gpu}"/>
 </robot>

Commit message: intrepid_description: add robot prefix_topic parameter to configure the ros namespace of intel D435 camera

File: intrepid_description/urdf/robots/intrepid.urdf.xacro (robot description, xacro)
@@ -48,6 +48,7 @@
     <xacro:property name="publish_bf" value="true" />
     <xacro:arg name="prefix" default="robot_" />
+    <xacro:arg name="prefix_topic" default="robot" />
     <xacro:property name="gpu" default="false" />
-    <xacro:macro name="intrepid" params="prefix publish_bf hq gpu">
+    <xacro:macro name="intrepid" params="prefix prefix_topic publish_bf hq gpu">
         <!-- *************** -->
         <!-- Robots Elements -->
@@ -102,8 +103,8 @@
  -->
         <!-- Kinova arm -->
-        <xacro:kinova_j2s6s200 parent="${prefix}base_link" x_position="${kinova_offset_x}" y_position="${kinova_offset_y}" z_position="${kinova_offset_z}"/>
+        <xacro:kinova_j2s6s200 parent="${prefix}base_link" x_position="${kinova_offset_x}" y_position="${kinova_offset_y}" z_position="${kinova_offset_z}" prefix_topic="${prefix_topic}"/>
     </xacro:macro>
     <!-- Gazebo ros control pluggins -->
     <xacro:ros_control/>
-    <xacro:intrepid prefix="$(arg prefix)" publish_bf="${publish_bf}" hq="${hq}" gpu="${gpu}"/>
+    <xacro:intrepid prefix="$(arg prefix)" prefix_topic="$(arg prefix_topic)" publish_bf="${publish_bf}" hq="${hq}" gpu="${gpu}"/>
 </robot>

File: intrepid_description/urdf/robots/j2s6s200_insert.xacro (robot description, xacro)
@@ -17,11 +17,11 @@
   <xacro:include filename="$(find intrepid_description)/urdf/structures/realsense2vgc10_support.urdf.xacro" />
   <xacro:include filename="$(find intrepid_description)/urdf/structures/intel_d435.urdf.xacro" />
-  <xacro:macro name="kinova_j2s6s200" params="parent x_position y_position z_position prefix:=j2s6s200">
+  <xacro:macro name="kinova_j2s6s200" params="parent x_position y_position z_position kinova_model:=j2s6s200 prefix_topic:=robot">
     <!-- Intel Realsense support-->
-    <xacro:realsense2vgc10_support prefix="${prefix}_wrist_rgbd_support" parent="${prefix}_link_5">
+    <xacro:realsense2vgc10_support prefix="${kinova_model}_wrist_rgbd_support" parent="${kinova_model}_link_5">
         <origin xyz="0.001 0.093 0.000" rpy="1.571 3.142 -3.142"/>
     </xacro:realsense2vgc10_support>
     <!-- Intel Realsense -->
-    <xacro:sensor_intel_d435 prefix="${prefix}_wrist_rgbd" parent="${prefix}_wrist_rgbd_support_second_link" prefix_topic="camera" use_nominal_extrinsics="true" >
+    <xacro:sensor_intel_d435 prefix="${kinova_model}_wrist_rgbd" parent="${kinova_model}_wrist_rgbd_support_second_link" prefix_topic="${prefix_topic}/camera" use_nominal_extrinsics="true" >
           <origin xyz="0.014 0.0 0.0" rpy="${pi} ${-pi/2} 0"/>
     </xacro:sensor_intel_d435>
